Commit message: feat(objects): reduced mass, friction for cabinet door

File: src/objects/collab_objects/cabinet.urdf (robot description, URDF)
Before this commit: robot cabinet, 11 links, 10 joints
Links:
- link door_handle: mass 0.1 -> 0.025

Commit message: feat(env): correct friction and actuation for robot

File: src/objects/collab_objects/cabinet.urdf (robot description, URDF)
Before this commit: robot cabinet, 11 links, 10 joints
Links:
- link door_handle: geometry collision box size=0.04 0.1 0.02; visual box size=0.04 0.1 0.02
