Commit message: fix(user_study): ready for user study (minus tasks desc)

File: src/objects/collab_objects/freezer.urdf (robot description, URDF)
Before this commit: robot freezer_top, 3 links, 2 joints
Links:
- link door_handle: mass None -> 0.1; geometry collision box size=0.025 0.011 0.1; visual box size=0.025 0.011 0.066
- link freezer_door: mass None -> 0.1; geometry collision box size=0.007 0.3 0.2; visual box size=0.007 0.3 0.2
Joints:
- joint handle_joint: origin xyz=0.015 0.27 0.1 -> xyz=0.025 0.27 0.1

File: src/objects/collab_objects/fridge.urdf (robot description, URDF)
Before this commit: robot fridge_bottom, 3 links, 2 joints
Links:
- link door_handle: mass None -> 0.1; geometry collision box size=0.025 0.011 0.1; visual box size=0.025 0.011 0.1
- link fridge_door: mass None -> 0.1
Joints:
- joint handle_joint: origin xyz=0.015 0.27 0.167 -> xyz=0.025 0.27 0.167
