Commit message: feature(objects): get robocasa objects handle, more realistic steak

File: src/objects/robocasa_objects/alborz_top_gas/alborz_top_gas.urdf (robot description, URDF)
Before this commit: robot alborz_top_gas, 6 links, 5 joints
Joints:
- joint knob_center_joint: limit lower=-3.1416 upper=3.1416 effort=1 velocity=0.1 -> lower=-3.1416 upper=3.1416 effort=1 velocity=0.0
- joint knob_front_left_joint: limit lower=-3.1416 upper=3.1416 effort=1 velocity=0.1 -> lower=-3.1416 upper=3.1416 effort=1 velocity=0.0
- joint knob_front_right_joint: limit lower=-3.1416 upper=3.1416 effort=1 velocity=0.1 -> lower=-3.1416 upper=3.1416 effort=1 velocity=0.0
- joint knob_rear_left_joint: limit lower=-3.1416 upper=3.1416 effort=1 velocity=0.1 -> lower=-3.1416 upper=3.1416 effort=1 velocity=0.0
- joint knob_rear_right_joint: limit lower=-3.1416 upper=3.1416 effort=1 velocity=0.1 -> lower=-3.1416 upper=3.1416 effort=1 velocity=0.0
